Commit message: [description] add primitive robot model, display launch and Blender bridge
- properties, inertial and material helpers (materials inline, safe to
  re-include from sensor xacros)
- chassis, wheels/caster, camera mast and gz DiffDrive/JointStatePublisher
  macros following INTERFACES.md sections 3-5 and 8
- display.launch.py with rviz/model.rviz for viewing the model without Gazebo
- local socket bridge to drive Blender from scripts (no external download)

Checked on Windows with xacro, flake8 and a static frame/size check;
not yet verified on Linux.

Co-Authored-By: Claude Opus 5.5 <noreply@anthropic.com>

File: src/serabot_description/urdf/camera_mast.xacro (robot description, xacro)
@@ -1,16 +1,36 @@
 <?xml version="1.0"?>
 <!--
-  PLACEHOLDER created by S0 so the top-level xacro builds.
-  Owner: S1 (robot model) - replace the macro body; keep the macro name and parameters
-  (they are part of the contract used by serabot.urdf.xacro).
+  SeraBot camera mast (owner: S1). Only the mounting post; the camera itself is
+  defined in sensors/camera.xacro on top of camera_mast_link (camera_z above it).
+  camera_mast_link sits at the foot of the mast, on the chassis top face.
+  Macro name and parameters are part of the contract (docs/INTERFACES.md section 8).
 -->
 <robot xmlns:xacro="http://www.ros.org/wiki/xacro">
+  <xacro:include filename="properties.xacro"/>
+  <xacro:include filename="materials.xacro"/>
+  <xacro:include filename="inertial_macros.xacro"/>
   <xacro:macro name="serabot_camera_mast">
     <joint name="camera_mast_joint" type="fixed">
       <parent link="base_link"/>
       <child link="camera_mast_link"/>
-      <origin xyz="-0.15 0 0.06" rpy="0 0 0"/>
+      <origin xyz="${mast_x} 0 ${mast_z}" rpy="0 0 0"/>
     </joint>
-    <link name="camera_mast_link"/>
+    <link name="camera_mast_link">
+      <visual>
+        <origin xyz="0 0 ${mast_height / 2}" rpy="0 0 0"/>
+        <geometry>
+          <cylinder radius="${mast_radius}" length="${mast_height}"/>
+        </geometry>
+        <xacro:serabot_material name="dark"/>
+      </visual>
+      <collision>
+        <origin xyz="0 0 ${mast_height / 2}" rpy="0 0 0"/>
+        <geometry>
+          <cylinder radius="${mast_radius}" length="${mast_height}"/>
+        </geometry>
+      </collision>
+      <xacro:inertial_cylinder mass="${mast_mass}" radius="${mast_radius}"
+                               length="${mast_height}" xyz="0 0 ${mast_height / 2}"/>
+    </link>
   </xacro:macro>
 </robot>

File: src/serabot_description/urdf/chassis.xacro (robot description, xacro)
@@ -1,9 +1,12 @@
 <?xml version="1.0"?>
 <!--
-  PLACEHOLDER created by S0 so the top-level xacro builds.
-  Owner: S1 (robot model) - replace the macro body; keep the macro name and parameters
-  (they are part of the contract used by serabot.urdf.xacro).
+  SeraBot chassis (owner: S1): base_footprint, base_link and the chassis body.
+  Macro name and parameters are part of the contract (docs/INTERFACES.md section 8).
+  Primitive visuals for now; they will be replaced by Blender meshes (ADR-012).
 -->
 <robot xmlns:xacro="http://www.ros.org/wiki/xacro">
+  <xacro:include filename="properties.xacro"/>
+  <xacro:include filename="materials.xacro"/>
+  <xacro:include filename="inertial_macros.xacro"/>
   <xacro:macro name="serabot_chassis">
     <link name="base_footprint"/>
@@ -11,7 +14,31 @@
       <parent link="base_footprint"/>
       <child link="base_link"/>
-      <origin xyz="0 0 0.08" rpy="0 0 0"/>
+      <origin xyz="0 0 ${base_height}" rpy="0 0 0"/>
     </joint>
-    <link name="base_link"/>
+    <link name="base_link">
+      <visual name="chassis_body">
+        <origin xyz="0 0 0" rpy="0 0 0"/>
+        <geometry>
+          <box size="${chassis_length} ${chassis_width} ${chassis_height}"/>
+        </geometry>
+        <xacro:serabot_material name="green"/>
+      </visual>
+      <visual name="front_bumper">
+        <origin xyz="${chassis_length / 2 - bumper_depth / 2 + bumper_protrusion} 0 ${bumper_z}"
+                rpy="0 0 0"/>
+        <geometry>
+          <box size="${bumper_depth} ${chassis_width + 2 * bumper_protrusion} ${bumper_height}"/>
+        </geometry>
+        <xacro:serabot_material name="terracotta"/>
+      </visual>
+      <collision>
+        <origin xyz="0 0 0" rpy="0 0 0"/>
+        <geometry>
+          <box size="${chassis_length} ${chassis_width} ${chassis_height}"/>
+        </geometry>
+      </collision>
+      <xacro:inertial_box mass="${chassis_mass}"
+                          x="${chassis_length}" y="${chassis_width}" z="${chassis_height}"/>
+    </link>
   </xacro:macro>
 </robot>

File: src/serabot_description/urdf/gazebo_drive.xacro (robot description, xacro)
@@ -1,10 +1,43 @@
 <?xml version="1.0"?>
 <!--
-  PLACEHOLDER created by S0 so the top-level xacro builds.
-  Owner: S1 (robot model) - replace the macro body; keep the macro name and parameters
-  (they are part of the contract used by serabot.urdf.xacro).
+  Gazebo (gz-sim) systems and surface friction for the SeraBot base (owner: S1).
+  DiffDrive and JointStatePublisher parameters follow docs/INTERFACES.md sections 2.1
+  and 5 (ADR-004). Macro name and parameters are part of the contract (section 8).
 -->
 <robot xmlns:xacro="http://www.ros.org/wiki/xacro">
+  <xacro:include filename="properties.xacro"/>
   <xacro:macro name="serabot_gazebo_drive">
+    <gazebo>
+      <plugin filename="gz-sim-diff-drive-system" name="gz::sim::systems::DiffDrive">
+        <left_joint>left_wheel_joint</left_joint>
+        <right_joint>right_wheel_joint</right_joint>
+        <wheel_separation>${wheel_separation}</wheel_separation>
+        <wheel_radius>${wheel_radius}</wheel_radius>
+        <max_linear_acceleration>${drive_max_linear_accel}</max_linear_acceleration>
+        <max_angular_acceleration>${drive_max_angular_accel}</max_angular_acceleration>
+        <topic>/cmd_vel</topic>
+        <odom_topic>/odom</odom_topic>
+        <tf_topic>/tf</tf_topic>
+        <frame_id>odom</frame_id>
+        <child_frame_id>base_footprint</child_frame_id>
+        <odom_publish_frequency>${drive_odom_rate}</odom_publish_frequency>
+      </plugin>
+      <plugin filename="gz-sim-joint-state-publisher-system"
+              name="gz::sim::systems::JointStatePublisher">
+        <topic>/joint_states</topic>
+      </plugin>
+    </gazebo>
+    <gazebo reference="left_wheel_link">
+      <mu1>${wheel_mu}</mu1>
+      <mu2>${wheel_mu}</mu2>
+    </gazebo>
+    <gazebo reference="right_wheel_link">
+      <mu1>${wheel_mu}</mu1>
+      <mu2>${wheel_mu}</mu2>
+    </gazebo>
+    <gazebo reference="caster_link">
+      <mu1>${caster_mu}</mu1>
+      <mu2>${caster_mu}</mu2>
+    </gazebo>
   </xacro:macro>
 </robot>

File: src/serabot_description/urdf/wheels.xacro (robot description, xacro)
@@ -1,10 +1,70 @@
 <?xml version="1.0"?>
 <!--
-  PLACEHOLDER created by S0 so the top-level xacro builds.
-  Owner: S1 (robot model) - replace the macro body; keep the macro name and parameters
-  (they are part of the contract used by serabot.urdf.xacro).
+  SeraBot drive wheels and caster (owner: S1).
+  Macro name and parameters are part of the contract (docs/INTERFACES.md section 8).
+  Wheel joints rotate about +Y, so a positive joint velocity drives the robot forward.
+  Friction settings live in gazebo_drive.xacro.
 -->
 <robot xmlns:xacro="http://www.ros.org/wiki/xacro">
+  <xacro:include filename="properties.xacro"/>
+  <xacro:include filename="materials.xacro"/>
+  <xacro:include filename="inertial_macros.xacro"/>
+  <!-- One drive wheel; side is "left" or "right", y_sign is +1 (left) or -1 (right). -->
+  <xacro:macro name="serabot_wheel" params="side y_sign">
+    <joint name="${side}_wheel_joint" type="continuous">
+      <parent link="base_link"/>
+      <child link="${side}_wheel_link"/>
+      <origin xyz="${wheel_x} ${y_sign * wheel_separation / 2} 0" rpy="0 0 0"/>
+      <axis xyz="0 1 0"/>
+    </joint>
+    <link name="${side}_wheel_link">
+      <visual name="tire">
+        <origin xyz="0 0 0" rpy="${pi / 2} 0 0"/>
+        <geometry>
+          <cylinder radius="${wheel_radius}" length="${wheel_width}"/>
+        </geometry>
+        <xacro:serabot_material name="rubber"/>
+      </visual>
+      <visual name="hub">
+        <origin xyz="0 ${y_sign * wheel_width / 4} 0" rpy="${pi / 2} 0 0"/>
+        <geometry>
+          <cylinder radius="${wheel_radius / 2}" length="${wheel_width / 2 + 0.002}"/>
+        </geometry>
+        <xacro:serabot_material name="terracotta"/>
+      </visual>
+      <collision>
+        <origin xyz="0 0 0" rpy="${pi / 2} 0 0"/>
+        <geometry>
+          <cylinder radius="${wheel_radius}" length="${wheel_width}"/>
+        </geometry>
+      </collision>
+      <xacro:inertial_cylinder mass="${wheel_mass}" radius="${wheel_radius}"
+                               length="${wheel_width}" rpy="${pi / 2} 0 0"/>
+    </link>
+  </xacro:macro>
   <xacro:macro name="serabot_wheels">
+    <xacro:serabot_wheel side="left" y_sign="1"/>
+    <xacro:serabot_wheel side="right" y_sign="-1"/>
+    <joint name="caster_joint" type="fixed">
+      <parent link="base_link"/>
+      <child link="caster_link"/>
+      <origin xyz="${caster_x} 0 ${caster_z}" rpy="0 0 0"/>
+    </joint>
+    <link name="caster_link">
+      <visual>
+        <origin xyz="0 0 0" rpy="0 0 0"/>
+        <geometry>
+          <sphere radius="${caster_radius}"/>
+        </geometry>
+        <xacro:serabot_material name="grey"/>
+      </visual>
+      <collision>
+        <origin xyz="0 0 0" rpy="0 0 0"/>
+        <geometry>
+          <sphere radius="${caster_radius}"/>
+        </geometry>
+      </collision>
+      <xacro:inertial_sphere mass="${caster_mass}" radius="${caster_radius}"/>
+    </link>
   </xacro:macro>
 </robot>

Commit message: [description] apply ADR-017 frames, hook up .obj meshes, sphere wheel collision
- base_link at the middle of the wheel axle (ADR-017): wheels x=0,
  chassis centre x=+0.12 (mesh offset via visual origin), caster +0.29,
  mast -0.03, lidar mount +0.22, imu 0; CoM x=+0.10 between axle and caster
- concept B meshes exported as .obj + .mtl (ADR-015) and used as visuals;
  use_mesh_visuals property switches back to the primitive visuals
- wheel collision is a sphere r=0.08: the cylinder touched the ground at its
  inner edge and /odom under-reported in-place rotation by 10.7 %; with the
  sphere it is 0.1 % (measured in Gazebo Jetty on the test VM)
- drop the .glb orientation test files, keep the primitive + .obj test
- report renders in docs/report/ (approved by the user)

Verified on the VM (Docker, Lyrical + Jetty 10.5.0): colcon build,
check_urdf, in-place rotation (footprint drift <= 0.7 mm) and straight drive.
RViz screenshot still pending (VM screen locked).

Co-Authored-By: Claude Opus 5.5 <noreply@anthropic.com>

File: src/serabot_description/urdf/camera_mast.xacro (robot description, xacro)
@@ -17,11 +17,21 @@
     </joint>
     <link name="camera_mast_link">
-      <visual>
-        <origin xyz="0 0 ${mast_height / 2}" rpy="0 0 0"/>
-        <geometry>
-          <cylinder radius="${mast_radius}" length="${mast_height}"/>
-        </geometry>
-        <xacro:serabot_material name="dark"/>
-      </visual>
+      <xacro:if value="${use_mesh_visuals}">
+        <visual>
+          <origin xyz="0 0 0" rpy="0 0 0"/>
+          <geometry>
+            <mesh filename="${mesh_dir}/camera_mast.obj"/>
+          </geometry>
+        </visual>
+      </xacro:if>
+      <xacro:unless value="${use_mesh_visuals}">
+        <visual>
+          <origin xyz="0 0 ${mast_height / 2}" rpy="0 0 0"/>
+          <geometry>
+            <cylinder radius="${mast_radius}" length="${mast_height}"/>
+          </geometry>
+          <xacro:serabot_material name="dark"/>
+        </visual>
+      </xacro:unless>
       <collision>
         <origin xyz="0 0 ${mast_height / 2}" rpy="0 0 0"/>

File: src/serabot_description/urdf/chassis.xacro (robot description, xacro)
@@ -3,5 +3,7 @@
   SeraBot chassis (owner: S1): base_footprint, base_link and the chassis body.
   Macro name and parameters are part of the contract (docs/INTERFACES.md section 8).
-  Primitive visuals for now; they will be replaced by Blender meshes (ADR-012).
+  base_link is the middle of the wheel axle (ADR-017); the chassis box is centred
+  chassis_x ahead of it. The chassis mesh is modelled around its own centre, so its
+  visual origin carries the same offset (INTERFACES.md section 4.1 exception).
 -->
 <robot xmlns:xacro="http://www.ros.org/wiki/xacro">
@@ -17,26 +19,36 @@
     </joint>
     <link name="base_link">
-      <visual name="chassis_body">
-        <origin xyz="0 0 0" rpy="0 0 0"/>
-        <geometry>
-          <box size="${chassis_length} ${chassis_width} ${chassis_height}"/>
-        </geometry>
-        <xacro:serabot_material name="green"/>
-      </visual>
-      <visual name="front_bumper">
-        <origin xyz="${chassis_length / 2 - bumper_depth / 2 + bumper_protrusion} 0 ${bumper_z}"
-                rpy="0 0 0"/>
-        <geometry>
-          <box size="${bumper_depth} ${chassis_width + 2 * bumper_protrusion} ${bumper_height}"/>
-        </geometry>
-        <xacro:serabot_material name="terracotta"/>
-      </visual>
+      <xacro:if value="${use_mesh_visuals}">
+        <visual name="chassis">
+          <origin xyz="${chassis_x} 0 0" rpy="0 0 0"/>
+          <geometry>
+            <mesh filename="${mesh_dir}/chassis.obj"/>
+          </geometry>
+        </visual>
+      </xacro:if>
+      <xacro:unless value="${use_mesh_visuals}">
+        <visual name="chassis_body">
+          <origin xyz="${chassis_x} 0 0" rpy="0 0 0"/>
+          <geometry>
+            <box size="${chassis_length} ${chassis_width} ${chassis_height}"/>
+          </geometry>
+          <xacro:serabot_material name="green"/>
+        </visual>
+        <visual name="front_bumper">
+          <origin xyz="${chassis_x + chassis_length / 2 - bumper_depth / 2 + bumper_protrusion} 0 ${bumper_z}"
+                  rpy="0 0 0"/>
+          <geometry>
+            <box size="${bumper_depth} ${chassis_width + 2 * bumper_protrusion} ${bumper_height}"/>
+          </geometry>
+          <xacro:serabot_material name="terracotta"/>
+        </visual>
+      </xacro:unless>
       <collision>
-        <origin xyz="0 0 0" rpy="0 0 0"/>
+        <origin xyz="${chassis_x} 0 0" rpy="0 0 0"/>
         <geometry>
           <box size="${chassis_length} ${chassis_width} ${chassis_height}"/>
         </geometry>
       </collision>
-      <xacro:inertial_box mass="${chassis_mass}"
+      <xacro:inertial_box mass="${chassis_mass}" xyz="${chassis_x} 0 0"
                           x="${chassis_length}" y="${chassis_width}" z="${chassis_height}"/>
     </link>

File: src/serabot_description/urdf/properties.xacro (robot description, xacro)
@@ -7,14 +7,21 @@
 -->
 <robot xmlns:xacro="http://www.ros.org/wiki/xacro">
-  <!-- Chassis box, centred on base_link (contract) -->
+  <!-- Visuals: Blender meshes (meshes/*.obj) or the primitive fallback (false), e.g. when
+       software rendering is too slow. Collisions are always primitives (ADR-012). -->
+  <xacro:property name="use_mesh_visuals" value="true"/>
+  <xacro:property name="mesh_dir" value="package://serabot_description/meshes"/>
+  <!-- base_link is the middle of the wheel axle at axle height; base_footprint is its
+       ground projection (contract, ADR-017). All x values below are from base_link. -->
+  <!-- Chassis box (contract); its centre is ahead of the axle -->
   <xacro:property name="chassis_length" value="0.45"/>
   <xacro:property name="chassis_width" value="0.30"/>
   <xacro:property name="chassis_height" value="0.12"/>
   <xacro:property name="chassis_mass" value="6.0"/>
+  <xacro:property name="chassis_x" value="0.12"/>
   <!-- Drive wheels (contract) -->
   <xacro:property name="wheel_radius" value="0.08"/>
   <xacro:property name="wheel_width" value="0.04"/>
   <xacro:property name="wheel_separation" value="0.36"/>
-  <xacro:property name="wheel_x" value="-0.12"/>
+  <xacro:property name="wheel_x" value="0.0"/>
   <xacro:property name="wheel_mass" value="0.5"/>
   <xacro:property name="wheel_mu" value="1.0"/>
@@ -23,10 +30,10 @@
   <!-- Frictionless caster sphere touching the ground (contract) -->
   <xacro:property name="caster_radius" value="0.03"/>
-  <xacro:property name="caster_x" value="0.17"/>
+  <xacro:property name="caster_x" value="0.29"/>
   <xacro:property name="caster_z" value="${caster_radius - base_height}"/>
   <xacro:property name="caster_mass" value="0.1"/>
   <xacro:property name="caster_mu" value="0.0"/>
   <!-- Camera mast, standing on the chassis top face (contract) -->
-  <xacro:property name="mast_x" value="-0.15"/>
+  <xacro:property name="mast_x" value="-0.03"/>
   <xacro:property name="mast_z" value="${chassis_height / 2}"/>
   <xacro:property name="mast_height" value="0.30"/>
@@ -39,5 +46,5 @@
   <xacro:property name="bumper_z" value="-0.02"/>
   <!-- Sensor mount points used by urdf/sensors/*.xacro (contract) -->
-  <xacro:property name="lidar_x" value="0.10"/>
+  <xacro:property name="lidar_x" value="0.22"/>
   <xacro:property name="lidar_y" value="0.0"/>
   <xacro:property name="lidar_z" value="0.10"/>

File: src/serabot_description/urdf/test/mesh_test.urdf.xacro (robot description, xacro)
@@ -2,10 +2,10 @@
 <!--
   Mesh orientation / colour test (owner: S1, ADR-015). Not part of the robot.
-  Four objects in a row along Y, each 0.1 m above the ground, should look identical:
+  Two objects in a row along Y, each 0.1 m above the ground, should look identical:
   grey cube, red arrow +X, green arrow +Y, blue cap +Z.
-    y = +0.6  ref_primitive  URDF primitives (ground truth)
-    y = +0.2  glb_yup        orientation_cube_yup.glb (glTF "+Y Up" export)
-    y = -0.2  glb_zup        orientation_cube_zup.glb (raw Blender axes)
-    y = -0.6  obj            orientation_cube.obj + .mtl
+    y = +0.3  ref_primitive  URDF primitives (ground truth)
+    y = -0.3  obj            orientation_cube.obj + .mtl (raw Blender axes)
+  Passed in RViz2 and Gazebo Jetty on 2026-10-24; the .glb variants were dropped
+  because the two tools apply the glTF axis conversion differently.
   RViz:   ros2 launch serabot_description display.launch.py model:=test/mesh_test.urdf.xacro
   Meshes: src/serabot_description/blender/make_orientation_test.py
@@ -41,5 +41,5 @@
   </xacro:macro>
   <link name="base_footprint"/>
-  <xacro:test_object name="ref_primitive" y="0.6">
+  <xacro:test_object name="ref_primitive" y="0.3">
     <visuals>
       <visual>
@@ -76,15 +76,5 @@
     </visuals>
   </xacro:test_object>
-  <xacro:test_object name="glb_yup" y="0.2">
-    <visuals>
-      <xacro:mesh_visual file="orientation_cube_yup.glb"/>
-    </visuals>
-  </xacro:test_object>
-  <xacro:test_object name="glb_zup" y="-0.2">
-    <visuals>
-      <xacro:mesh_visual file="orientation_cube_zup.glb"/>
-    </visuals>
-  </xacro:test_object>
-  <xacro:test_object name="obj" y="-0.6">
+  <xacro:test_object name="obj" y="-0.3">
     <visuals>
       <xacro:mesh_visual file="orientation_cube.obj"/>

File: src/serabot_description/urdf/wheels.xacro (robot description, xacro)
@@ -19,22 +19,36 @@
     </joint>
     <link name="${side}_wheel_link">
-      <visual name="tire">
-        <origin xyz="0 0 0" rpy="${pi / 2} 0 0"/>
+      <xacro:if value="${use_mesh_visuals}">
+        <!-- Symmetric mesh, axle along Y: the same file serves both sides -->
+        <visual name="wheel">
+          <origin xyz="0 0 0" rpy="0 0 0"/>
+          <geometry>
+            <mesh filename="${mesh_dir}/wheel.obj"/>
+          </geometry>
+        </visual>
+      </xacro:if>
+      <xacro:unless value="${use_mesh_visuals}">
+        <visual name="tire">
+          <origin xyz="0 0 0" rpy="${pi / 2} 0 0"/>
+          <geometry>
+            <cylinder radius="${wheel_radius}" length="${wheel_width}"/>
+          </geometry>
+          <xacro:serabot_material name="rubber"/>
+        </visual>
+        <visual name="hub">
+          <origin xyz="0 ${y_sign * wheel_width / 4} 0" rpy="${pi / 2} 0 0"/>
+          <geometry>
+            <cylinder radius="${wheel_radius / 2}" length="${wheel_width / 2 + 0.002}"/>
+          </geometry>
+          <xacro:serabot_material name="terracotta"/>
+        </visual>
+      </xacro:unless>
+      <!-- Sphere, not cylinder: a cylinder touches the ground at its inner edge, which
+           shrinks the effective track (~0.325 m) and made /odom under-report in-place
+           rotation by ~11 %; the sphere's single contact keeps it at wheel_separation. -->
+      <collision>
+        <origin xyz="0 0 0" rpy="0 0 0"/>
         <geometry>
-          <cylinder radius="${wheel_radius}" length="${wheel_width}"/>
-        </geometry>
-        <xacro:serabot_material name="rubber"/>
-      </visual>
-      <visual name="hub">
-        <origin xyz="0 ${y_sign * wheel_width / 4} 0" rpy="${pi / 2} 0 0"/>
-        <geometry>
-          <cylinder radius="${wheel_radius / 2}" length="${wheel_width / 2 + 0.002}"/>
-        </geometry>
-        <xacro:serabot_material name="terracotta"/>
-      </visual>
-      <collision>
-        <origin xyz="0 0 0" rpy="${pi / 2} 0 0"/>
-        <geometry>
-          <cylinder radius="${wheel_radius}" length="${wheel_width}"/>
+          <sphere radius="${wheel_radius}"/>
         </geometry>
       </collision>
@@ -55,7 +69,14 @@
         <origin xyz="0 0 0" rpy="0 0 0"/>
         <geometry>
-          <sphere radius="${caster_radius}"/>
+          <xacro:if value="${use_mesh_visuals}">
+            <mesh filename="${mesh_dir}/caster.obj"/>
+          </xacro:if>
+          <xacro:unless value="${use_mesh_visuals}">
+            <sphere radius="${caster_radius}"/>
+          </xacro:unless>
         </geometry>
-        <xacro:serabot_material name="grey"/>
+        <xacro:unless value="${use_mesh_visuals}">
+          <xacro:serabot_material name="grey"/>
+        </xacro:unless>
       </visual>
       <collision>
