Commit message: [description] add RViz/Gazebo mesh colour sets and gazebo_mesh_colors arg
RViz2 reads MTL diffuse colours as display (sRGB) values while Gazebo
Jetty treats them as linear, so one MTL cannot look right in both.

- meshes/*.mtl now hold sRGB colours (RViz2); meshes/gazebo/ has the same
  OBJ files with Blender's linear colours (Gazebo)
- properties.xacro: xacro arg gazebo_mesh_colors (default false) selects
  mesh_dir; the URDF spawned in Gazebo should be generated with it set
- mesh_kit.export_obj writes both sets; the test cube MTL uses sRGB too

Checked on the test VM: build, check_urdf with the arg, RViz and Gazebo
screenshots show the intended colours.

Co-Authored-By: Claude Opus 5.5 <noreply@anthropic.com>

File: src/serabot_description/urdf/properties.xacro (robot description, xacro)
@@ -10,5 +10,15 @@
        software rendering is too slow. Collisions are always primitives (ADR-012). -->
   <xacro:property name="use_mesh_visuals" value="true"/>
-  <xacro:property name="mesh_dir" value="package://serabot_description/meshes"/>
+  <!-- Mesh colour set. RViz2 reads MTL colours as display (sRGB) values, Gazebo Jetty as
+       linear ones, so meshes/ holds sRGB MTLs and meshes/gazebo/ the same OBJs with linear
+       MTLs. Generate the URDF that is spawned in Gazebo with gazebo_mesh_colors:=true;
+       robot_state_publisher / RViz keep the default. -->
+  <xacro:arg name="gazebo_mesh_colors" default="false"/>
+  <xacro:if value="$(arg gazebo_mesh_colors)">
+    <xacro:property name="mesh_dir" value="package://serabot_description/meshes/gazebo"/>
+  </xacro:if>
+  <xacro:unless value="$(arg gazebo_mesh_colors)">
+    <xacro:property name="mesh_dir" value="package://serabot_description/meshes"/>
+  </xacro:unless>
   <!-- base_link is the middle of the wheel axle at axle height; base_footprint is its
        ground projection (contract, ADR-017). All x values below are from base_link. -->
