Commit message: [lidar] add gpu_lidar sensor macro and bridge config
lidar_link with the pebble mesh, cylinder collision and inertial on
lidar_joint (properties.xacro mount point); gpu_lidar on /scan, 360
samples, 10 Hz, 0.25-8.0 m, gaussian noise. Verified on the VM.

Co-Authored-By: Claude Opus 5.5 <noreply@anthropic.com>

File: src/serabot_description/urdf/sensors/lidar.xacro (robot description, xacro)
@@ -1,10 +1,99 @@
 <?xml version="1.0"?>
 <!--
-  PLACEHOLDER created by S0 so the top-level xacro builds.
-  Owner: Member A (LiDAR) - replace the macro body; keep the macro name and parameters
-  (they are part of the contract used by serabot.urdf.xacro).
+  SeraBot 2D LiDAR (owner: Member A). docs/INTERFACES.md sections 2.2, 3, 4 and 8.
+  lidar_link is the scan centre: lidar_x/y/z above base_link from properties.xacro.
+  The scan plane is 0.18 m above the ground, so it clears the chassis top (0.14 m)
+  and hits walls (1.0 m), plant beds (0.40 m) and pots (0.35 m). The pebble mesh
+  and the camera mast (0.235 m away) lie inside range_min, so the robot does not
+  see itself. Macro name and parameter are part of the contract.
 -->
 <robot xmlns:xacro="http://www.ros.org/wiki/xacro">
+  <xacro:include filename="../properties.xacro"/>
+  <xacro:include filename="../materials.xacro"/>
+  <xacro:include filename="../inertial_macros.xacro"/>
+  <!-- Housing: bounding cylinder of meshes/lidar.obj (r 0.042, z -0.05 .. +0.01) -->
+  <xacro:property name="lidar_body_radius" value="0.042"/>
+  <xacro:property name="lidar_body_height" value="0.06"/>
+  <xacro:property name="lidar_body_z" value="-0.02"/>
+  <xacro:property name="lidar_mass" value="0.15"/>
+  <!-- Sensor settings (contract, INTERFACES.md section 2.2) -->
+  <xacro:property name="lidar_topic" value="scan"/>
+  <xacro:property name="lidar_rate" value="10"/>
+  <xacro:property name="lidar_samples" value="360"/>
+  <xacro:property name="lidar_min_angle" value="${-pi}"/>
+  <xacro:property name="lidar_max_angle" value="${pi}"/>
+  <xacro:property name="lidar_range_min" value="0.25"/>
+  <xacro:property name="lidar_range_max" value="8.0"/>
+  <xacro:property name="lidar_range_resolution" value="0.01"/>
+  <xacro:property name="lidar_noise_stddev" value="0.01"/>
   <xacro:macro name="serabot_lidar" params="parent">
+    <joint name="lidar_joint" type="fixed">
+      <parent link="${parent}"/>
+      <child link="lidar_link"/>
+      <origin xyz="${lidar_x} ${lidar_y} ${lidar_z}" rpy="0 0 0"/>
+    </joint>
+    <link name="lidar_link">
+      <xacro:if value="${use_mesh_visuals}">
+        <visual>
+          <origin xyz="0 0 0" rpy="0 0 0"/>
+          <geometry>
+            <mesh filename="${mesh_dir}/lidar.obj"/>
+          </geometry>
+        </visual>
+      </xacro:if>
+      <xacro:unless value="${use_mesh_visuals}">
+        <visual>
+          <origin xyz="0 0 ${lidar_body_z}" rpy="0 0 0"/>
+          <geometry>
+            <cylinder radius="${lidar_body_radius}" length="${lidar_body_height}"/>
+          </geometry>
+          <xacro:serabot_material name="dark"/>
+        </visual>
+      </xacro:unless>
+      <collision>
+        <origin xyz="0 0 ${lidar_body_z}" rpy="0 0 0"/>
+        <geometry>
+          <cylinder radius="${lidar_body_radius}" length="${lidar_body_height}"/>
+        </geometry>
+      </collision>
+      <xacro:inertial_cylinder mass="${lidar_mass}" radius="${lidar_body_radius}"
+                               length="${lidar_body_height}" xyz="0 0 ${lidar_body_z}"/>
+    </link>
+    <gazebo reference="lidar_link">
+      <sensor name="lidar" type="gpu_lidar">
+        <pose>0 0 0 0 0 0</pose>
+        <topic>${lidar_topic}</topic>
+        <gz_frame_id>lidar_link</gz_frame_id>
+        <update_rate>${lidar_rate}</update_rate>
+        <always_on>true</always_on>
+        <visualize>false</visualize>
+        <lidar>
+          <scan>
+            <horizontal>
+              <samples>${lidar_samples}</samples>
+              <resolution>1</resolution>
+              <min_angle>${lidar_min_angle}</min_angle>
+              <max_angle>${lidar_max_angle}</max_angle>
+            </horizontal>
+            <vertical>
+              <samples>1</samples>
+              <resolution>1</resolution>
+              <min_angle>0</min_angle>
+              <max_angle>0</max_angle>
+            </vertical>
+          </scan>
+          <range>
+            <min>${lidar_range_min}</min>
+            <max>${lidar_range_max}</max>
+            <resolution>${lidar_range_resolution}</resolution>
+          </range>
+          <noise>
+            <type>gaussian</type>
+            <mean>0.0</mean>
+            <stddev>${lidar_noise_stddev}</stddev>
+          </noise>
+        </lidar>
+      </sensor>
+    </gazebo>
   </xacro:macro>
 </robot>
